File: BenchBudEE/Power.sch (KiCad schematic (older format))
At the start: 0 parts

Commit message: Roughly populated the Power sheet.
Parts:
- added C? (x2): C, ~, symbol C
- added F? (x4): FUSE, ~, symbol FUSE
- added L? (x2): INDUCTOR, ~, symbol INDUCTOR
- added P?: CONN_12X2, symbol CONN_12X2
- added R?: R, ~, symbol R
- added SW?: SWITCH_INV, ~, symbol SWITCH_INV
Connections:
- new net: F?.1, P?.10 (P10)
- new net: F?.1, P?.14 (P14)
- new net: P?.16 (P16), SW?.2
- new net: F?.1, P?.2 (P2)
- new net: F?.1, P?.4 (P4), P?.6 (P6)
- new net: R?.1, SW?.1
- new net +12P: F?.2, L?.1
- new net +12V: C?.1, L?.2
- new net +3.3V: F?.2, R?.2
- new net +5V: F?.2
- new net -12P: F?.2, L?.1
- new net -12V: C?.2, L?.2
- new net GND: C?.1, C?.2, P?.3 (P3), P?.5 (P5), SW?.3
Other:
- note added: "ATX Power Supply - Molex 24-pin"
- note added: "Filter"
- note added: "Fuses might be PTC Thermistors"

Commit message: Revisiting the current/fan module.
Parts:
- removed F? (x4): FUSE, ~, symbol FUSE
- added TH? (x4): THERMISTOR, ~, symbol THERMISTOR
Connections:
- net +12P: now also TH?.2
- net +3.3V: now also TH?.2
- net +5V: now also TH?.2
- net -12P: now also TH?.2
- net +12C: now reaches P?.10 (P10)
- net +12C: now also TH?.1
- net at P?.14 (P14): now also TH?.1
- net at P?.2 (P2): now also TH?.1
- net at P?.4 (P4), P?.6 (P6): now also TH?.1
Other:
- note added: "PTC Thermistors to limit current"
- note removed: "Fuses might be PTC Thermistors"
Changed lines of the file:
@@
 $Descr A4 11693 8268
 encoding utf-8
-Sheet 5 9
+Sheet 4 9
 Title ""
-Date "10 feb 2014"
+Date "12 feb 2014"
 Rev ""
 Comp ""
@@
 	1    0    0    -1
 $EndComp
-Connection ~ 3450 1600
-Connection ~ 1650 1250
 Wire Wire Line
 	2950 1500 3450 1500
@@
 Wire Wire Line
 	3250 3150 3550 3150
-Text Notes 1850 1150 0    60   ~ 0
+Text Notes 1250 1100 0    60   ~ 0
 ATX Power Supply - Molex 24-pin
 Connection ~ 10300 1900
@@
 Text Notes 9650 1200 0    60   ~ 0
 Filter
-Text Notes 5000 2300 0    60   ~ 0
-Fuses might be PTC Thermistors
+Text Notes 3950 2350 0    60   ~ 0
+PTC Thermistors to limit current
 $Comp
 L GND #PWR?
@@
 $EndComp
 $Comp
-L FUSE F?
-U 1 1 52F629E9
-P 5700 2100
-F 0 "F?" H 5800 2150 40  0000 C CNN
-F 1 "FUSE" H 5600 2050 40  0000 C CNN
-F 2 "~" H 5700 2100 60  0000 C CNN
-F 3 "~" H 5700 2100 60  0000 C CNN
-	1    5700 2100
-	1    0    0    -1
-$EndComp
-$Comp
-L FUSE F?
-U 1 1 52F629E3
-P 5150 1900
-F 0 "F?" H 5250 1950 40  0000 C CNN
-F 1 "FUSE" H 5050 1850 40  0000 C CNN
-F 2 "~" H 5150 1900 60  0000 C CNN
-F 3 "~" H 5150 1900 60  0000 C CNN
-	1    5150 1900
-	1    0    0    -1
-$EndComp
-$Comp
-L FUSE F?
-U 1 1 52F629DD
-P 4400 1700
-F 0 "F?" H 4500 1750 40  0000 C CNN
-F 1 "FUSE" H 4300 1650 40  0000 C CNN
-F 2 "~" H 4400 1700 60  0000 C CNN
-F 3 "~" H 4400 1700 60  0000 C CNN
-	1    4400 1700
-	1    0    0    -1
-$EndComp
-$Comp
-L FUSE F?
-U 1 1 52F629C6
-P 3700 1500
-F 0 "F?" H 3800 1550 40  0000 C CNN
-F 1 "FUSE" H 3600 1450 40  0000 C CNN
-F 2 "~" H 3700 1500 60  0000 C CNN
-F 3 "~" H 3700 1500 60  0000 C CNN
-	1    3700 1500
-	1    0    0    -1
-$EndComp
-$Comp
 L +5V #PWR?
 U 1 1 52F62810
@@
 	1    0    0    -1
 $EndComp
+Wire Wire Line
+	3300 1900 3300 1050
+Connection ~ 3300 1900
+$Comp
+L +12C #PWR?
+U 1 1 52FAE7F5
+P 3300 1050
+F 0 "#PWR?" H 3300 1020 30  0001 C CNN
+F 1 "+12C" H 3300 1160 40  0000 C CNN
+F 2 "" H 3300 1050 60  0000 C CNN
+F 3 "" H 3300 1050 60  0000 C CNN
+	1    3300 1050
+	1    0    0    -1
+$EndComp
+$Comp
+L THERMISTOR TH?
+U 1 1 52FB015D
+P 3700 1500
+F 0 "TH?" V 3800 1550 50  0000 C CNN
+F 1 "THERMISTOR" V 3600 1500 50  0000 C CNN
+F 2 "~" H 3700 1500 60  0000 C CNN
+F 3 "~" H 3700 1500 60  0000 C CNN
+	1    3700 1500
+	0    -1   -1   0
+$EndComp
+$Comp
+L THERMISTOR TH?
+U 1 1 52FB016A
+P 4400 1700
+F 0 "TH?" V 4500 1750 50  0000 C CNN
+F 1 "THERMISTOR" V 4300 1700 50  0000 C CNN
+F 2 "~" H 4400 1700 60  0000 C CNN
+F 3 "~" H 4400 1700 60  0000 C CNN
+	1    4400 1700
+	0    -1   -1   0
+$EndComp
+$Comp
+L THERMISTOR TH?
+U 1 1 52FB0170
+P 5150 1900
+F 0 "TH?" V 5250 1950 50  0000 C CNN
+F 1 "THERMISTOR" V 5050 1900 50  0000 C CNN
+F 2 "~" H 5150 1900 60  0000 C CNN
+F 3 "~" H 5150 1900 60  0000 C CNN
+	1    5150 1900
+	0    -1   -1   0
+$EndComp
+$Comp
+L THERMISTOR TH?
+U 1 1 52FB0180
+P 5700 2100
+F 0 "TH?" V 5800 2150 50  0000 C CNN
+F 1 "THERMISTOR" V 5600 2100 50  0000 C CNN
+F 2 "~" H 5700 2100 60  0000 C CNN
+F 3 "~" H 5700 2100 60  0000 C CNN
+	1    5700 2100
+	0    -1   -1   0
+$EndComp
 $EndSCHEMATC
