File: BenchBudEE/Relay.sch (KiCad schematic (older format))
At the start: 11 parts

Commit message: Placed the relay components.
Parts:
- removed R?: R, ~, symbol R
- removed U?: PHTRANS, ~, symbol PHTRANS
- added R5: 0, ~, symbol R
- added U1: LTV-816S, symbol OPTO-TRANSISTOR4
- D1: renamed from D?; value LED -> LG Q971-KN-1
- D2: renamed from D?; value DIODE -> B130-13-F
- K1: renamed from K?; value SPDT -> 1461069-5
- Q1: renamed from Q?; value NPN -> 2N3904; MFG Name (none) -> Diodes Inc; MFG Part Number (none) -> MMBT3904-7-F
- R1: renamed from R?; value R -> 500
- R2: renamed from R?; value R -> 200
- R3, R6: renamed from R?; value R -> 0
- R4: renamed from R?; value R -> 100
Other:
- note added: "1V Drop"
- note added: "2V CE Drop"
- note added: "2V Drop"
- note added: "DIODE SCHOTTKY 30V 1A SMA"
- note added: "LED CHIPLED 570NM GREEN 0603 SMD"
- note added: "OPTOCOUPLER TRANS 5KVRMS 4SMD"
- note added: "RELAY GEN PURPOSE SPDT 10A 12V"
- note added: "TRANS NPN 40V 350MW SMD SOT23-3"
- note removed: "Relay"
- moved on the sheet: R1
Changed lines of the file:
@@
 $Descr A4 11693 8268
 encoding utf-8
-Sheet 4 9
+Sheet 3 9
 Title ""
-Date "19 feb 2014"
+Date "20 feb 2014"
 Rev ""
 Comp ""
@@
 Comment4 ""
 $EndDescr
-Text HLabel 1850 4150 0    60   Input ~ 0
+Text HLabel 1750 4250 0    60   Input ~ 0
 RELAY+
-Text HLabel 1850 4500 0    60   Output ~ 0
+Text HLabel 1750 4550 0    60   Output ~ 0
 RELAY-
 Text HLabel 9900 3200 2    60   BiDi ~ 0
@@
 RELAY_NO
 $Comp
-L PHTRANS U?
-U 1 1 52F440BD
-P 3800 4350
-F 0 "U?" H 3750 4700 70  0000 C CNN
-F 1 "PHTRANS" H 3750 4000 70  0000 C CNN
-F 2 "~" H 3800 4350 60  0000 C CNN
-F 3 "~" H 3800 4350 60  0000 C CNN
-	1    3800 4350
-	1    0    0    -1
-$EndComp
-$Comp
-L R R?
+L R R4
 U 1 1 52F440DB
 P 5750 4550
-F 0 "R?" V 5830 4550 40  0000 C CNN
-F 1 "R" V 5757 4551 40  0000 C CNN
+F 0 "R4" V 5830 4550 40  0000 C CNN
+F 1 "100" V 5757 4551 40  0000 C CNN
 F 2 "~" V 5680 4550 30  0000 C CNN
 F 3 "~" H 5750 4550 30  0000 C CNN
@@
 $EndComp
 $Comp
-L NPN Q?
+L NPN Q1
 U 1 1 52F440EA
 P 7950 4550
-F 0 "Q?" H 7950 4400 50  0000 R CNN
-F 1 "NPN" H 7950 4700 50  0000 R CNN
+F 0 "Q1" H 7950 4400 50  0000 R CNN
+F 1 "2N3904" H 7950 4700 50  0000 R CNN
 F 2 "~" H 7950 4550 60  0000 C CNN
 F 3 "~" H 7950 4550 60  0000 C CNN
+F 4 "Diodes Inc" H 7950 4550 60  0001 C CNN "MFG Name"
+F 5 "MMBT3904-7-F" H 7950 4550 60  0001 C CNN "MFG Part Number"
 	1    7950 4550
 	1    0    0    -1
 $EndComp
 $Comp
-L LED D?
+L LED D1
 U 1 1 52F440F9
 P 5300 5200
-F 0 "D?" H 5300 5300 50  0000 C CNN
-F 1 "LED" H 5300 5100 50  0000 C CNN
+F 0 "D1" H 5300 5300 50  0000 C CNN
+F 1 "LG Q971-KN-1" H 5300 5100 50  0000 C CNN
 F 2 "~" H 5300 5200 60  0000 C CNN
 F 3 "~" H 5300 5200 60  0000 C CNN
@@
 $EndComp
 $Comp
-L SPDT K?
+L SPDT K1
 U 1 1 52F44639
 P 8650 3250
-F 0 "K?" H 8650 3500 70  0000 C CNN
-F 1 "SPDT" H 8650 2650 70  0000 C CNN
+F 0 "K1" H 8650 3500 70  0000 C CNN
+F 1 "1461069-5" H 8650 2650 70  0000 C CNN
 F 2 "~" H 8650 3250 60  0000 C CNN
 F 3 "~" H 8650 3250 60  0000 C CNN
@@
 	9050 3400 9900 3400
 Wire Wire Line
-	4350 4550 5500 4550
+	4200 4550 5500 4550
 Wire Wire Line
 	6000 4550 7750 4550
 Wire Wire Line
-	5500 3500 8250 3500
-Wire Wire Line
 	8050 4750 8050 5300
 $Comp
-L R R?
+L R R6
 U 1 1 52F448EE
 P 8050 5550
-F 0 "R?" V 8130 5550 40  0000 C CNN
-F 1 "R" V 8057 5551 40  0000 C CNN
+F 0 "R6" V 8130 5550 40  0000 C CNN
+F 1 "0" V 8057 5551 40  0000 C CNN
 F 2 "~" V 7980 5550 30  0000 C CNN
 F 3 "~" H 8050 5550 30  0000 C CNN
@@
 $EndComp
 $Comp
-L GND #PWR?
+L GND #PWR12
 U 1 1 52F448F6
 P 8050 6150
-F 0 "#PWR?" H 8050 6150 30  0001 C CNN
+F 0 "#PWR12" H 8050 6150 30  0001 C CNN
 F 1 "GND" H 8050 6080 30  0001 C CNN
 F 2 "" H 8050 6150 60  0000 C CNN
@@
 	8050 5800 8050 6150
 Wire Wire Line
-	5500 2900 5500 4350
-Wire Wire Line
 	5300 5000 5300 4550
 Connection ~ 5300 4550
 $Comp
-L R R?
+L R R2
 U 1 1 52F44A66
 P 5300 5750
-F 0 "R?" V 5380 5750 40  0000 C CNN
-F 1 "R" V 5307 5751 40  0000 C CNN
+F 0 "R2" V 5380 5750 40  0000 C CNN
+F 1 "200" V 5307 5751 40  0000 C CNN
 F 2 "~" V 5230 5750 30  0000 C CNN
 F 3 "~" H 5300 5750 30  0000 C CNN
@@
 	5300 6000 8050 6000
 Connection ~ 8050 6000
-$Comp
-L R R?
-U 1 1 52F44A89
-P 5500 2650
-F 0 "R?" V 5580 2650 40  0000 C CNN
-F 1 "R" V 5507 2651 40  0000 C CNN
-F 2 "~" V 5430 2650 30  0000 C CNN
-F 3 "~" H 5500 2650 30  0000 C CNN
-	1    5500 2650
-	-1   0    0    1
-$EndComp
 Wire Wire Line
 	5500 1900 5500 2400
-Wire Wire Line
-	5500 4350 4350 4350
-Connection ~ 5500 3500
-$Comp
-L R R?
-U 1 1 52F44ACB
-P 4950 4150
-F 0 "R?" V 5030 4150 40  0000 C CNN
-F 1 "R" V 4957 4151 40  0000 C CNN
-F 2 "~" V 4880 4150 30  0000 C CNN
-F 3 "~" H 4950 4150 30  0000 C CNN
-	1    4950 4150
+$Comp
+L R R1
+U 1 1 52F44AFE
+P 2450 4550
+F 0 "R1" V 2530 4550 40  0000 C CNN
+F 1 "500" V 2457 4551 40  0000 C CNN
+F 2 "~" V 2380 4550 30  0000 C CNN
+F 3 "~" H 2450 4550 30  0000 C CNN
+	1    2450 4550
 	0    1    1    0
 $EndComp
 Wire Wire Line
-	4350 4150 4700 4150
-Wire Wire Line
-	5200 4150 5500 4150
-Connection ~ 5500 4150
-$Comp
-L R R?
-U 1 1 52F44AFE
-P 2550 4500
-F 0 "R?" V 2630 4500 40  0000 C CNN
-F 1 "R" V 2557 4501 40  0000 C CNN
-F 2 "~" V 2480 4500 30  0000 C CNN
-F 3 "~" H 2550 4500 30  0000 C CNN
-	1    2550 4500
-	0    1    1    0
-$EndComp
-Wire Wire Line
-	2800 4500 3250 4500
-Wire Wire Line
-	1850 4500 2300 4500
-Wire Wire Line
-	1850 4150 3250 4150
+	1750 4550 2200 4550
 Wire Wire Line
 	9950 2550 8150 2550
@@
 	8150 3300 8250 3300
 Wire Wire Line
-	8050 4350 8050 3600
+	8050 3600 8050 4350
 Wire Wire Line
 	8050 3600 8250 3600
 $Comp
-L DIODE D?
+L DIODE D2
 U 1 1 52F44F61
 P 7500 3900
-F 0 "D?" H 7500 4000 40  0000 C CNN
-F 1 "DIODE" H 7500 3800 40  0000 C CNN
+F 0 "D2" H 7500 4000 40  0000 C CNN
+F 1 "B130-13-F" H 7500 3800 40  0000 C CNN
 F 2 "~" H 7500 3900 60  0000 C CNN
 F 3 "~" H 7500 3900 60  0000 C CNN
@@
 $EndComp
 Wire Wire Line
-	7500 3700 7500 3500
+	7500 2900 7500 3700
 Connection ~ 7500 3500
 Wire Wire Line
@@
 Text Notes 6600 3950 0    60   ~ 0
 Kickback Diode
-Text Notes 9000 4000 0    60   ~ 0
-Relay
-$Comp
-L +12P #PWR?
+$Comp
+L +12P #PWR11
 U 1 1 52F62CEB
 P 5500 1900
-F 0 "#PWR?" H 5500 1870 30  0001 C CNN
+F 0 "#PWR11" H 5500 1870 30  0001 C CNN
 F 1 "+12P" H 5500 2000 30  0000 C CNN
 F 2 "" H 5500 1900 60  0000 C CNN
@@
 	1    0    0    -1
 $EndComp
+$Comp
+L OPTO-TRANSISTOR4 U1
+U 1 1 5305DFF2
+P 3600 4400
+F 0 "U1" H 3800 4650 60  0000 C CNN
+F 1 "LTV-816S" H 3600 4150 60  0000 C CNN
+F 2 "" H 3600 4400 60  0000 C CNN
+F 3 "" H 3600 4400 60  0000 C CNN
+F 4 "LTV-816S" H 3600 4400 60  0001 C CNN "MFG Part Number"
+	1    3600 4400
+	1    0    0    -1
+$EndComp
+Wire Wire Line
+	2700 4550 2950 4550
+Wire Wire Line
+	1750 4250 2950 4250
+Wire Wire Line
+	5500 4250 4200 4250
+Connection ~ 5500 4250
+Wire Wire Line
+	5500 2900 5500 4250
+Text Notes 5500 5250 0    60   ~ 0
+LED CHIPLED 570NM GREEN 0603 SMD
+Text Notes 6050 4100 0    60   ~ 0
+DIODE SCHOTTKY 30V 1A SMA
+Text Notes 2850 4850 0    60   ~ 0
+OPTOCOUPLER TRANS 5KVRMS 4SMD
+Text Notes 8250 4600 0    60   ~ 0
+TRANS NPN 40V 350MW SMD SOT23-3
+Text Notes 8350 4050 0    60   ~ 0
+RELAY GEN PURPOSE SPDT 10A 12V
+Text Notes 4100 4450 0    60   ~ 0
+2V CE Drop
+Wire Wire Line
+	7500 3500 8250 3500
+$Comp
+L R R5
+U 1 1 5305F4BB
+P 7500 2650
+F 0 "R5" V 7580 2650 40  0000 C CNN
+F 1 "0" V 7507 2651 40  0000 C CNN
+F 2 "~" V 7430 2650 30  0000 C CNN
+F 3 "~" H 7500 2650 30  0000 C CNN
+	1    7500 2650
+	-1   0    0    1
+$EndComp
+Wire Wire Line
+	7500 2400 7500 2100
+Wire Wire Line
+	7500 2100 5500 2100
+Connection ~ 5500 2100
+$Comp
+L R R3
+U 1 1 52F44A89
+P 5500 2650
+F 0 "R3" V 5580 2650 40  0000 C CNN
+F 1 "0" V 5507 2651 40  0000 C CNN
+F 2 "~" V 5430 2650 30  0000 C CNN
+F 3 "~" H 5500 2650 30  0000 C CNN
+	1    5500 2650
+	-1   0    0    1
+$EndComp
+Text Notes 4650 5250 0    60   ~ 0
+1V Drop
+Text Notes 2850 4400 0    60   ~ 0
+2V Drop
 $EndSCHEMATC
